File: WT32-ETH01 WLED CTRL.kicad_sch (KiCad schematic)
At the start: 20 parts, among them J1 USB_C_Receptacle_USB2.0_14P, Q1 S8050, Q2 S8050, SW1 Reset, SW2 Boot, U1 WT32-ETH01, U2 CH340C

Commit message: Updated Board to REV2.0 - Removed usb reset circut - Added antenna cutout - Added TX/RX LEDs
Parts:
- removed C4, C5: 100nF, Capacitor_SMD:C_0805_2012Metric_Pad1.18x1.45mm_HandSolder, symbol Device:C_Small
- removed Q1, Q2: S8050, Package_TO_SOT_SMD:SOT-23_Handsoldering, symbol Transistor_BJT:S8050
- added D1: RXD, LED_SMD:LED_0805_2012Metric, symbol Device:LED
- added D2: TXD, LED_SMD:LED_0805_2012Metric, symbol Device:LED
- added F1: Fuse, Fuse:Fuse_0805_2012Metric_Pad1.15x1.40mm_HandSolder, symbol Device:Fuse
- R1, R2: value 10k -> 330; LCSC Part # (none) -> C17630
Connections:
- net +5V: now also R1.1, R2.1, F1.2; no longer J1.A4 (VBUS), J1.A9 (VBUS), J1.B4 (VBUS), J1.B9 (VBUS)
- net RXD: now also R4.1, U2.2 (TXD), D1.1 (K); no longer R4.2, U1.25 (IO3/PRG_RX)
- net TXD: now also R3.1, U2.3 (RXD), D2.1 (K); no longer R3.2, U1.26 (IO1/PRG_TX)
- net DTR: no longer names the net of R1.2
- net DTR: now also D1.2 (A); no longer U2.13 (~{DTR})
- net RTS: no longer names the net of U2.14 (~{RTS})
- net RTS: no longer R2.2
- new net: D2.2 (A), R2.2
- new net MCU_RXD: R4.2, U1.25 (IO3/PRG_RX)
- new net MCU_TXD: R3.2, U1.26 (IO1/PRG_TX)
- new net VBUS: F1.1, J1.A4 (VBUS), J1.A9 (VBUS), J1.B4 (VBUS), J1.B9 (VBUS)
- no-connect marks 19 -> 21
Other:
- moved on the sheet: R3, R4
